File: fra_clock.kicad_pcb (KiCad board)
At the start: 2 copper layers, 210 x 297 mm, 425 parts, among them J1 USB_C, J101 SPK_TOP, J102 SPK_BOT, Q1 MMBT3904, Q2 MMBT3904, Q3 2N7002, U1 AP2112K-3.3, U101 MAX98357A, U102 MAX98357A, U2 USBLC6-2SC6, U3 ESP32-WROOM-32E, U5 CH340C, U6 74AHCT125

Commit message: Phase A: critical routing (CRITICAL_AUTO) - power, USB, audio outputs, GND vias
DRC A: 0 errors besides unconnected Phase-B nets; warnings: 14 pre-existing lib_footprint_mismatch, 4 dangling LED_x_DIN vias (Phase B).

Co-Authored-By: Claude Opus 5.5 <noreply@anthropic.com>
Claude-Session: https://claude.ai/code/session_01UYk7fLNsQphaXPRGVQJ5XY
Routing:
- net +5V: track 1416.8 -> 1837.5 mm, vias 3 -> 11
- net +3V3: track 0.00 -> 158.2 mm, vias 0 -> 2
- net /USB_DM: track 0.00 -> 97.0 mm, vias 0 -> 2
- net /USB_DP: track 0.00 -> 94.0 mm
- net GND: track 363.6 -> 432.5 mm, vias 360 -> 402
- net /VBUS: track 0.00 -> 25.8 mm, vias 0 -> 5
- net Net-(J102-Pin_2): track 0.00 -> 20.9 mm
- net Net-(J101-Pin_2): track 0.00 -> 20.9 mm
- net Net-(J102-Pin_1): track 0.00 -> 15.6 mm
- net Net-(J101-Pin_1): track 0.00 -> 15.6 mm
- net Net-(J1-CC2): track 0.00 -> 6.62 mm, vias 0 -> 2
- net Net-(J1-CC1): track 0.00 -> 5.80 mm, vias 0 -> 2

Commit message: Phase B: Freerouting 2.5.0 + scripted fixes (FREEROUTE_AUTO), GND plane continuity
DRC B: 0 errors, 0 unconnected, 0 schematic parity issues; only 14 pre-existing lib_footprint_mismatch warnings.
Phase A updated: J1 GND ties, U6 GND spine, C69.2 tie.

Co-Authored-By: Claude Opus 5.5 <noreply@anthropic.com>
Claude-Session: https://claude.ai/code/session_01UYk7fLNsQphaXPRGVQJ5XY
Routing:
- net /AUD_DIN: track 0.00 -> 413.7 mm, vias 0 -> 7
- net /AMP_SHDN: track 0.00 -> 398.8 mm, vias 0 -> 3
- net /AUD_WS: track 0.00 -> 383.6 mm, vias 0 -> 3
- net /AUD_BCLK: track 0.00 -> 367.6 mm, vias 0 -> 5
- net /LED_C_DIN: track 1.20 -> 312.2 mm, vias 1 -> 6
- net /LED_B_DIN: track 1.20 -> 252.7 mm, vias 1 -> 2
- net /LED_D_DIN: track 1.20 -> 226.5 mm, vias 1 -> 2
- net /ESP_TX: track 0.00 -> 192.1 mm, vias 0 -> 6
- net /ESP_IO0: track 0.00 -> 177.8 mm, vias 0 -> 2
- net /ESP_RX: track 0.00 -> 177.4 mm, vias 0 -> 6
- net /ESP_EN: track 0.00 -> 173.6 mm, vias 0 -> 2
- net /LED_A_3V3: track 0.00 -> 108.4 mm, vias 0 -> 4
- net /LED_B_3V3: track 0.00 -> 99.0 mm, vias 0 -> 4
- net /LED_C_3V3: track 0.00 -> 89.1 mm
- net +3V3: track 158.2 -> 224.7 mm, vias 2 -> 4
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